File: pcb/chuckplus.kicad_pcb (KiCad board)
At the start: 2 copper layers, 229.7 x 114.9 mm, 83 parts

Commit message: chuck plus with rkjxt encoder
Parts:
- added SW35: , ComboDiode, B.Cu at (151.9, 97.7)
- added SW36: , ComboDiode, B.Cu at (151.9, 94.7)
- added SW37: , ComboDiode, B.Cu at (151.9, 91.7)
- added SW38: , pts526, B.Cu at (171.9, 47.7)
- ENC1: footprint ceoloide:rotary_encoder_ec11_ec12 -> Alps_Alpine_RKJXT
- SW34: footprint pts526 -> ComboDiode
- moved SW34 56.6 mm to (151.9, 100.7)
- moved SW33 2.00 mm to (151.9, 103.7)
Connections:
- ENC1 pad A: ENC_A -> rkjxt_A
- ENC1 pad B: ENC_B -> rkjxt_B
- ENC1 pad C: GND -> rkjxt_C
- SW33 pad 1: D7 -> D13
- SW33 pad 2: encdiode -> rkjxt_A
- SW34 pad 1: GND -> D14
- SW34 pad 2: RST -> rkjxt_B
Routing:
- net D4: track 250.3 -> 298.6 mm, vias 1 -> 4
- net D17: track 119.3 -> 167.0 mm
- net D6: track 119.7 -> 165.2 mm, vias 2 -> 0
- net D15: track 102.2 -> 143.5 mm, vias 1 -> 0
- net rkjxt_PUSH: track 0.00 -> 34.7 mm
- net rkjxt_D: track 0.00 -> 26.1 mm
- net rkjxt_A: track 0.00 -> 21.9 mm
- net rkjxt_B: track 0.00 -> 19.0 mm
- net D14: track 142.6 -> 161.5 mm, vias 1 -> 2
- net D13: track 162.2 -> 181.1 mm, vias 2 -> 0
- net D19: track 173.7 -> 157.6 mm, vias 1 -> 2
- net BAT+: track 38.7 -> 53.3 mm
- net rkjxt_C: track 0.00 -> 11.6 mm
- net D3: track 349.5 -> 360.2 mm
- net ENC_B: track 72.9 -> 62.8 mm
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Other:
- rule pad_to_mask_clearance: 0.05 -> 0
- board text removed: "D4-D7"

Commit message: v4 with xiao nrf52840 plus, rkjxt and hardware debounce
Parts:
- added ?: , MountingHole_2.2mm_M2_Pad_Via, F.Cu at (151.9, 77.7)
- added ?: , MountingHole_2.2mm_M2_Pad_Via, F.Cu at (114.8, 39.9)
- added ?: , MountingHole_2.2mm_M2_Pad_Via, F.Cu at (189.0, 39.9)
- added DB1: , Smd0805, B.Cu at (164.9, 52.7)
- added DB2: , Smd0805, B.Cu at (164.9, 55.7)
- added DB3: , Smd0805, B.Cu at (164.9, 61.7)
- added DB4: , Smd0805, B.Cu at (164.9, 64.7)
- added DB5: , Smd0805, B.Cu at (164.9, 67.7)
- added DB6: , Smd0805, B.Cu at (164.9, 73.7)
- added DB7: , ComboDiode, B.Cu at (164.9, 58.7)
- added DB8: , ComboDiode, B.Cu at (164.9, 70.7)
Connections:
- ? pad D8: ENC_B -> B_DB
- ? pad D9: ENC_A -> A_DB
- ENC1 pad COM: D4 -> D10
Routing:
- net GND: track 137.9 -> 10.6 mm, vias 0 -> 4
- net D10: track 0.00 -> 67.5 mm, vias 0 -> 4
- net D6: track 165.2 -> 118.7 mm, vias 0 -> 2
- net VCC: track 0.00 -> 42.9 mm, vias 0 -> 2
- net ENC_A: track 71.5 -> 95.5 mm
- net B_DB: track 0.00 -> 22.8 mm
- net D7: track 171.2 -> 190.0 mm, vias 1 -> 2
- net D17: track 167.0 -> 148.4 mm, vias 1 -> 2
- net D4: track 298.6 -> 281.2 mm, vias 4 -> 2
- net A_DB: track 0.00 -> 16.0 mm
- net ENC_B: track 62.8 -> 49.6 mm
- net D2: track 420.1 -> 430.3 mm
- net D3: track 360.2 -> 352.2 mm
- net BAT+: track 53.3 -> 61.2 mm, vias 0 -> 2
- net D19: track 157.6 -> 164.4 mm
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Other:
- rule pad_to_mask_clearance: 0 -> 0.05
